File: EAGLE/Quad_Cape.brd (EAGLE design)
At the start: 55.3 x 35.3 mm, 24 parts, among them IC1 TPD4S012DRY, U1 POCKETBEAGLE, U2 MS5611-01BA03, U3 ICM-20948, U4 TXS0102DQER

Commit message: Final changes for V1 board
Parts:
- added FUD1, FUD2, FUD3: FIDUCIAL, Quad_Cape:FIDUCIAL_40MIL
- added U$5: (no value), Strawson_Eagle_Lib:XYZ_BIG
- X1: value (none) -> USB
- moved R4 8.84 mm to (17.0, 26.0), turned to 0 degrees
- moved R3 6.55 mm to (17.7, 19.4), turned to 180 degrees
- moved R5 0.25 mm to (21.5, 26.0)
Connections:
- removed net VIN.USB: C5.1, IC1.6, X1.1
- net USBC.D+: now also IC1.2; no longer IC1.1
- net USBC.D-: now also IC1.1; no longer IC1.2
- net USB_DC: now also C5.1, IC1.6, X1.1
Routing:
- net USBC.D+: track 68.3 -> 56.9 mm
- net GND: track 37.6 -> 27.2 mm, vias 13 -> 14
- net VIN.USB: track 8.06 -> 0.00 mm
- net N$2: track 7.17 -> 1.68 mm
- net VDD_3P3V: track 13.3 -> 10.1 mm, vias 7 -> 8
- net MOTOR2: track 24.6 -> 23.5 mm
- net USBC.D-: track 55.4 -> 56.5 mm
- net MOTOR4: track 25.7 -> 24.7 mm
- net USB_DC: track 2.54 -> 1.79 mm, vias 0 -> 1
- net IMU_SCL: track 15.4 -> 14.8 mm
- net VDD_1P8V: track 11.8 -> 11.3 mm
- net GPS_TX: track 13.5 -> 14.0 mm
- added copper zone on layer 16, net USB_DC
Other:
- board text added: "Quad Cape V1"
- board text added: "W Grimes"
