File: EAGLE/Quad_Cape.sch (EAGLE design)
At the start: 24 parts, among them IC1 TPD4S012DRY, U1 POCKETBEAGLE, U2 MS5611-01BA03, U3 ICM-20948, U4 TXS0102DQER

Commit message: Final changes for V1 board
Parts:
- added FUD1, FUD2, FUD3: FIDUCIAL, Quad_Cape:FIDUCIAL
- X1: value (none) -> USB
Connections:
- removed net VIN.USB: C5.1, IC1.VBUS, X1.VBUS
- net USBC.D+: now also IC1.D-; no longer IC1.D+
- net USBC.D-: now also IC1.D+; no longer IC1.D-
- net USB_DC: now also C5.1, IC1.VBUS, X1.VBUS
Other:
- note added: "ACCEL/GYRO (W/ LVL. SHFT. 3.3V to 1.8V)"
- note added: "MECHANICAL"
- note added: "Note: the +/- pins for the ESD protection are interchangeable"
- note removed: "ACCEROMETER/GYROSCOPE (W/ LVL. SHFT. 3.3V to 1.8V)"
Changed lines of the file:
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@@
 <part name="SUPPLY7" library="ENGI301" deviceset="VDD_3P3V" device=""/>
 <part name="SUPPLY10" library="ENGI301" deviceset="VDD_3P3V" device=""/>
-<part name="SUPPLY13" library="GHI-PowerGoundSupply" deviceset="USB_DC" device="" value="VIN.USB"/>
 <part name="IC1" library="GHI-IC" deviceset="TPD4S012DRYR" device="" value="TPD4S012DRY"/>
 <part name="GND15" library="supply1" library_urn="urn:adsk.eagle:library:371" deviceset="GND" device=""/>
 <part name="C5" library="GHI-BasicComponents" deviceset="CAPACITOR-(INCH)-" device="0402" value=".1uF"/>
-<part name="SUPPLY2" library="GHI-PowerGoundSupply" deviceset="USB_DC" device="" value="VIN.USB"/>
-<part name="X1" library="Quad_Cape" deviceset="GHI2_USB_HOST_W/CHASSIS_GND" device=""/>
+<part name="X1" library="Quad_Cape" deviceset="GHI2_USB_HOST_W/CHASSIS_GND" device="" value="USB"/>
 <part name="GND12" library="supply1" library_urn="urn:adsk.eagle:library:371" deviceset="GND" device=""/>
 <part name="SUPPLY3" library="Quad_Cape" deviceset="VDD_1P8V" device=""/>
@@
 <part name="H1" library="Quad_Cape" deviceset="3PIN_100MIL" device=""/>
 <part name="GND4" library="Quad_Cape" deviceset="GND" device=""/>
+<part name="FUD1" library="Quad_Cape" deviceset="FIDUCIAL" device=""/>
+<part name="FUD2" library="Quad_Cape" deviceset="FIDUCIAL" device=""/>
+<part name="FUD3" library="Quad_Cape" deviceset="FIDUCIAL" device=""/>
+<part name="SUPPLY4" library="Quad_Cape" deviceset="USB_DC" device=""/>
+<part name="SUPPLY2" library="Quad_Cape" deviceset="USB_DC" device=""/>
 </parts>
 <sheets>
@@
 <wire x1="530.86" y1="558.8" x2="530.86" y2="490.22" width="0.1524" layer="97"/>
 <wire x1="530.86" y1="490.22" x2="530.86" y2="386.08" width="0.1524" layer="97"/>
-<wire x1="530.86" y1="386.08" x2="530.86" y2="314.96" width="0.1524" layer="97"/>
+<wire x1="530.86" y1="386.08" x2="530.86" y2="342.9" width="0.1524" layer="97"/>
+<wire x1="530.86" y1="342.9" x2="530.86" y2="314.96" width="0.1524" layer="97"/>
 <wire x1="530.86" y1="386.08" x2="581.66" y2="386.08" width="0.1524" layer="97"/>
 <wire x1="581.66" y1="386.08" x2="772.16" y2="386.08" width="0.1524" layer="97"/>
@@
 <text x="535.94" y="558.8" size="5.08" layer="97" rot="MR180">BAROMETER/ALTIMETER</text>
 <text x="670.56" y="551.18" size="5.08" layer="97">USB</text>
-<text x="586.74" y="477.52" size="5.08" layer="97">ACCEROMETER/GYROSCOPE (W/ LVL. SHFT. 3.3V to 1.8V)</text>
+<text x="584.2" y="477.52" size="5.08" layer="97">ACCEL/GYRO (W/ LVL. SHFT. 3.3V to 1.8V)</text>
 <text x="436.88" y="533.4" size="5.08" layer="97">POCKET BEAGLE</text>
 <text x="718.82" y="309.88" size="2.1844" layer="94">1 of 1</text>
 <wire x1="581.66" y1="490.22" x2="581.66" y2="386.08" width="0.1524" layer="97"/>
 <text x="541.02" y="477.52" size="5.08" layer="97">POWER IN</text>
+<wire x1="401.32" y1="342.9" x2="530.86" y2="342.9" width="0.1524" layer="97"/>
+<text x="452.12" y="335.28" size="2.54" layer="97">MECHANICAL</text>
+<text x="706.12" y="495.3" size="1.778" layer="97">Note: the +/- pins for the ESD protection are interchangeable</text>
 </plain>
 <instances>
@@
 <attribute name="VALUE" x="612.14" y="550.164" size="1.778" layer="96" align="center"/>
 </instance>
-<instance part="SUPPLY13" gate="G$1" x="746.76" y="530.86" smashed="yes">
-<attribute name="VALUE" x="746.76" y="534.924" size="1.778" layer="96" align="center"/>
-</instance>
 <instance part="IC1" gate="G$1" x="731.52" y="508" smashed="yes">
 <attribute name="NAME" x="723.9" y="513.842" size="1.016" layer="95" ratio="12"/>
@@
 <attribute name="VALUE" x="749.554" y="505.968" size="1.778" layer="96"/>
 </instance>
-<instance part="SUPPLY2" gate="G$1" x="424.18" y="416.56" smashed="yes">
-<attribute name="VALUE" x="424.18" y="420.624" size="1.778" layer="96" align="center"/>
-</instance>
 <instance part="X1" gate="G$1" x="690.88" y="520.7" smashed="yes" rot="R270">
 <attribute name="NAME" x="703.58" y="533.4" size="1.27" layer="95" rot="R270"/>
@@
 <instance part="GND4" gate="1" x="568.96" y="424.18" smashed="yes">
 <attribute name="VALUE" x="566.42" y="421.64" size="1.778" layer="96"/>
+</instance>
+<instance part="FUD1" gate="G$1" x="454.66" y="325.12" smashed="yes"/>
+<instance part="FUD2" gate="G$1" x="462.28" y="325.12" smashed="yes"/>
+<instance part="FUD3" gate="G$1" x="469.9" y="325.12" smashed="yes"/>
+<instance part="SUPPLY4" gate="G$1" x="746.76" y="530.86" smashed="yes">
+<attribute name="VALUE" x="746.76" y="534.924" size="1.778" layer="96" align="center"/>
+</instance>
+<instance part="SUPPLY2" gate="G$1" x="424.18" y="416.56" smashed="yes">
+<attribute name="VALUE" x="424.18" y="420.624" size="1.778" layer="96" align="center"/>
 </instance>
 </instances>
@@
 </segment>
 </net>
-<net name="VIN.USB" class="0">
-<segment>
-<pinref part="SUPPLY13" gate="G$1" pin="USB_DC"/>
+<net name="USBC.D-" class="0">
+<segment>
+<pinref part="U1" gate="G$1" pin="USB1.D-"/>
+<wire x1="441.96" y1="406.4" x2="424.18" y2="406.4" width="0.1524" layer="91"/>
+<label x="424.18" y="406.4" size="1.778" layer="95"/>
+</segment>
+<segment>
+<label x="716.28" y="523.24" size="1.778" layer="95"/>
+<pinref part="IC1" gate="G$1" pin="D+"/>
+<wire x1="721.36" y1="510.54" x2="713.74" y2="510.54" width="0.1524" layer="91"/>
+<wire x1="713.74" y1="510.54" x2="713.74" y2="523.24" width="0.1524" layer="91"/>
+<wire x1="713.74" y1="523.24" x2="726.44" y2="523.24" width="0.1524" layer="91"/>
+<pinref part="X1" gate="G$1" pin="D-"/>
+<wire x1="713.74" y1="523.24" x2="703.58" y2="523.24" width="0.1524" layer="91"/>
+<junction x="713.74" y="523.24"/>
+</segment>
+</net>
+<net name="USBC.D+" class="0">
+<segment>
+<pinref part="U1" gate="G$1" pin="USB1.D+"/>
+<wire x1="441.96" y1="403.86" x2="424.18" y2="403.86" width="0.1524" layer="91"/>
+<label x="424.18" y="403.86" size="1.778" layer="95"/>
+</segment>
+<segment>
+<wire x1="726.44" y1="520.7" x2="711.2" y2="520.7" width="0.1524" layer="91"/>
+<label x="716.28" y="520.7" size="1.778" layer="95"/>
+<pinref part="IC1" gate="G$1" pin="D-"/>
+<wire x1="721.36" y1="508" x2="711.2" y2="508" width="0.1524" layer="91"/>
+<wire x1="711.2" y1="508" x2="711.2" y2="520.7" width="0.1524" layer="91"/>
+<pinref part="X1" gate="G$1" pin="D+"/>
+<wire x1="711.2" y1="520.7" x2="703.58" y2="520.7" width="0.1524" layer="91"/>
+<junction x="711.2" y="520.7"/>
+</segment>
+</net>
+<net name="USB_DC" class="0">
+<segment>
 <pinref part="IC1" gate="G$1" pin="VBUS"/>
 <wire x1="741.68" y1="510.54" x2="746.76" y2="510.54" width="0.1524" layer="91"/>
@@
 <pinref part="C5" gate="G$1" pin="1"/>
 <pinref part="X1" gate="G$1" pin="VBUS"/>
-</segment>
-</net>
-<net name="USBC.D-" class="0">
-<segment>
-<pinref part="U1" gate="G$1" pin="USB1.D-"/>
-<wire x1="441.96" y1="406.4" x2="424.18" y2="406.4" width="0.1524" layer="91"/>
-<label x="424.18" y="406.4" size="1.778" layer="95"/>
-</segment>
-<segment>
-<wire x1="726.44" y1="523.24" x2="711.2" y2="523.24" width="0.1524" layer="91"/>
-<label x="716.28" y="523.24" size="1.778" layer="95"/>
-<pinref part="IC1" gate="G$1" pin="D-"/>
-<wire x1="711.2" y1="523.24" x2="703.58" y2="523.24" width="0.1524" layer="91"/>
-<wire x1="721.36" y1="508" x2="711.2" y2="508" width="0.1524" layer="91"/>
-<wire x1="711.2" y1="508" x2="711.2" y2="523.24" width="0.1524" layer="91"/>
-<junction x="711.2" y="523.24"/>
-<pinref part="X1" gate="G$1" pin="D-"/>
-</segment>
-</net>
-<net name="USBC.D+" class="0">
-<segment>
-<pinref part="U1" gate="G$1" pin="USB1.D+"/>
-<wire x1="441.96" y1="403.86" x2="424.18" y2="403.86" width="0.1524" layer="91"/>
-<label x="424.18" y="403.86" size="1.778" layer="95"/>
-</segment>
-<segment>
-<label x="716.28" y="520.7" size="1.778" layer="95"/>
-<pinref part="IC1" gate="G$1" pin="D+"/>
-<wire x1="713.74" y1="520.7" x2="703.58" y2="520.7" width="0.1524" layer="91"/>
-<wire x1="721.36" y1="510.54" x2="713.74" y2="510.54" width="0.1524" layer="91"/>
-<wire x1="713.74" y1="510.54" x2="713.74" y2="520.7" width="0.1524" layer="91"/>
-<pinref part="X1" gate="G$1" pin="D+"/>
-<wire x1="713.74" y1="520.7" x2="726.44" y2="520.7" width="0.1524" layer="91"/>
-<junction x="713.74" y="520.7"/>
-</segment>
-</net>
-<net name="USB_DC" class="0">
+<pinref part="SUPPLY4" gate="G$1" pin="USB_DC"/>
+</segment>
 <segment>
 <pinref part="U1" gate="G$1" pin="USB1.VIN"/>
 <wire x1="441.96" y1="408.94" x2="424.18" y2="408.94" width="0.1524" layer="91"/>
 <wire x1="424.18" y1="408.94" x2="424.18" y2="411.48" width="0.1524" layer="91"/>
-<pinref part="SUPPLY2" gate="G$1" pin="USB_DC"/>
 <pinref part="U1" gate="G$1" pin="USB1.VBUS"/>
 <wire x1="424.18" y1="411.48" x2="424.18" y2="414.02" width="0.1524" layer="91"/>
 <wire x1="441.96" y1="411.48" x2="424.18" y2="411.48" width="0.1524" layer="91"/>
 <junction x="424.18" y="411.48"/>
+<pinref part="SUPPLY2" gate="G$1" pin="USB_DC"/>
 </segment>
 </net>
@@
 </sheet>
 </sheets>
+<errors>
+</errors>
 </schematic>
 </drawing>
